Commit message: Bruh

File: ros_ws/src/litevla_bridge/resource/litevla_robot.urdf (robot description, URDF)
Before this commit: robot litevla_robot, 0 links, 0 joints
Links:
- added link base_link
- added link left_wheel
- added link right_wheel
Joints:
- added joint left wheel motor: type continuous, parent base_link, child left_wheel, origin xyz=0 0.03 0 rpy=0 0 0, axis 0 1 0
- added joint right wheel motor: type continuous, parent base_link, child right_wheel, origin xyz=0 -0.03 0 rpy=0 0 0, axis 0 1 0

Commit message: Bruh

File: ros_ws/src/litevla_bridge/resource/litevla_robot.urdf (robot description, URDF)
Before this commit: robot litevla_robot, 3 links, 2 joints
Joints:
- joint left wheel motor: origin xyz=0 0.03 0 rpy=0 0 0 -> xyz=0 0.03 0.02 rpy=0 0 0
- joint right wheel motor: origin xyz=0 -0.03 0 rpy=0 0 0 -> xyz=0 -0.03 0.02 rpy=0 0 0
