Commit message: Add Epic 105 dataset pipeline on Raj/VLA-06-code-only branch.
Port dataset schema, builder, validator, loader, labeling, and sim capture
from Raj/VLA-06 while preserving current main Epic 103/104 modules.

Co-authored-by: Cursor <cursoragent@cursor.com>

File: ros_ws/src/litevla_bridge/resource/litevla_robot.urdf (robot description, URDF)
Before this commit: robot litevla_robot, 0 links, 0 joints
Links:
- added link base_link
- added link left_wheel
- added link right_wheel
Joints:
- added joint left wheel motor: type continuous, parent base_link, child left_wheel, origin xyz=0 0.03 0.02 rpy=0 0 0, axis 0 1 0
- added joint right wheel motor: type continuous, parent base_link, child right_wheel, origin xyz=0 -0.03 0.02 rpy=0 0 0, axis 0 1 0
